File: pcb/arena-clock/auxillary_sr.kicad_sch (KiCad schematic)
At the start: 2 parts, among them U10 TPIC6595

Commit message: Update kicad schematic and layout with metadata (release date, title, company) and export pdfs as sent to mfg on 11/19.
Other:
- company: (none) -> MassDestruction (Sarah Pohorecky)
- title: (none) -> Arena Clock Carrier
Changed lines of the file:
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@@
 (kicad_sch (version 20211123) (generator eeschema)
   (paper "A4")
+  (title_block
+    (title "Arena Clock Carrier")
+    (date "2023-11-19")
+    (rev "1.0")
+    (company "MassDestruction (Sarah Pohorecky)")
+  )
   (no_connect (at 118.11 97.79))
   (bus_entry (at 151.13 95.25) (size 2.54 2.54)
