File: pcb/arena-clock/board_output.kicad_sch (KiCad schematic)
At the start: 72 parts, among them J1 SPEAKER ENABLE, J10 Conn_01x03_Male, J11 12V POW CONN, J12 5V POW CONN, J13 AUX SINK, J14 AUX GPIO, J2 DIGIT1, J3 DIGIT2, J4 DIGIT3, J5 DIGIT4, J6 DIGIT5, J7 DIGIT6, J8 AUX 12V OUT, J9 Conn_01x03_Male, U4 J107F1CS1212VDC.36, U5 J107F1CS1212VDC.36

Commit message: Update kicad schematic and layout with metadata (release date, title, company) and export pdfs as sent to mfg on 11/19.
Other:
- company: (none) -> MassDestruction (Sarah Pohorecky)
- title: (none) -> Arena Clock Carrier
Changed lines of the file:
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@@
 (kicad_sch (version 20211123) (generator eeschema)
   (paper "A4")
+  (title_block
+    (title "Arena Clock Carrier")
+    (date "2023-11-19")
+    (rev "1.0")
+    (company "MassDestruction (Sarah Pohorecky)")
+  )
   (junction (at 246.38 41.91) (diameter 0) (color 0 0 0 0)
   )
