File: pcb/arena-clock/digit_display.kicad_sch (KiCad schematic)
At the start: 6 parts, among them U1 TPIC6595, U2 TPIC6595, U3 TPIC6595

Commit message: Update kicad schematic and layout with metadata (release date, title, company) and export pdfs as sent to mfg on 11/19.
Other:
- company: (none) -> MassDestruction (Sarah Pohorecky)
- title: (none) -> Arena Clock Carrier
Changed lines of the file:
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@@
 (kicad_sch (version 20211123) (generator eeschema)
   (paper "A4")
+  (title_block
+    (title "Arena Clock Carrier")
+    (date "2023-11-19")
+    (rev "1.0")
+    (company "MassDestruction (Sarah Pohorecky)")
+  )
   (bus_alias "DIGIT5" (members "_0" "_1"))
   (no_connect (at 49.53 160.02))
