File: pcb/arena-clock/level_shifters.kicad_sch (KiCad schematic)
At the start: 6 parts, among them U11 TXU0104, U12 TXU0104

Commit message: Update kicad schematic and layout with metadata (release date, title, company) and export pdfs as sent to mfg on 11/19.
Other:
- company: (none) -> MassDestruction (Sarah Pohorecky)
- title: (none) -> Arena Clock Carrier
Changed lines of the file:
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@@
 (kicad_sch (version 20211123) (generator eeschema)
   (paper "A4")
+  (title_block
+    (title "Arena Clock Carrier")
+    (date "2023-11-19")
+    (rev "1.0")
+    (company "MassDestruction (Sarah Pohorecky)")
+  )
   (bus_entry (at 158.75 96.52) (size -2.54 2.54)
     (stroke (width 0) (type default) (color 0 0 0 0))
