File: pcb/arena-clock/onboard_display.kicad_sch (KiCad schematic)
At the start: 27 parts, among them U6 HDSP-7501, U7 HDSP-7501, U8 HDSP-7501

Commit message: Update kicad schematic and layout with metadata (release date, title, company) and export pdfs as sent to mfg on 11/19.
Other:
- company: (none) -> MassDestruction (Sarah Pohorecky)
- title: (none) -> Arena Clock Carrier
Changed lines of the file:
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@@
 (kicad_sch (version 20211123) (generator eeschema)
   (paper "A4")
+  (title_block
+    (title "Arena Clock Carrier")
+    (date "2023-11-19")
+    (rev "1.0")
+    (company "MassDestruction (Sarah Pohorecky)")
+  )
   (junction (at 102.87 53.34) (diameter 0) (color 0 0 0 0)
   )
