File: pcb/arena-clock/stm32_headers.kicad_sch (KiCad schematic)
At the start: 4 parts, among them J16 CN3 Breakout, J17 CN3, J18 CN4, J19 CN4 Breakout

Commit message: Update kicad schematic and layout with metadata (release date, title, company) and export pdfs as sent to mfg on 11/19.
Other:
- company: (none) -> MassDestruction (Sarah Pohorecky)
- title: (none) -> Arena Clock Carrier
Changed lines of the file:
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@@
 (kicad_sch (version 20211123) (generator eeschema)
   (paper "A4")
+  (title_block
+    (title "Arena Clock Carrier")
+    (date "2023-11-19")
+    (rev "1.0")
+    (company "MassDestruction (Sarah Pohorecky)")
+  )
   (junction (at 91.44 93.98) (diameter 0) (color 0 0 0 0)
   )
